File: pcb/USB-C-2.0.kicad_sch (KiCad schematic)
At the start: 4 parts, among them J18 USB_C_Receptacle_USB2.0_16P, U25 ESD73034D-10/TR(ES)

Commit message: fixed schematic
Parts:
- renumbered J18 to J6, R93 to R37, R94 to R38, U25 to U8
Changed lines of the file:
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@@
 		(dnp no)
 		(fields_autoplaced yes)
-		(property "Reference" "J18"
+		(property "Reference" "J6"
 			(at 132.08 60.96 0)
 			(show_name no)
@@
 			(project "pcb"
 				(path "/124991ae-9d31-41fe-b759-30be3a40922b/a13fb698-9f77-4d73-8ccf-806a48de5dab"
-					(reference "J18")
+					(reference "J6")
 					(unit 1)
 				)
@@
 		(dnp no)
 		(fields_autoplaced yes)
-		(property "Reference" "R94"
+		(property "Reference" "R38"
 			(at 170.18 68.58 0)
 			(show_name no)
@@
 			(project "pcb"
 				(path "/124991ae-9d31-41fe-b759-30be3a40922b/a13fb698-9f77-4d73-8ccf-806a48de5dab"
-					(reference "R94")
+					(reference "R38")
 					(unit 1)
 				)
@@
 		(in_pos_files yes)
 		(dnp no)
-		(property "Reference" "U25"
+		(property "Reference" "U8"
 			(at 167.64 80.01 0)
 			(show_name no)
@@
 			(project "pcb"
 				(path "/124991ae-9d31-41fe-b759-30be3a40922b/a13fb698-9f77-4d73-8ccf-806a48de5dab"
-					(reference "U25")
+					(reference "U8")
 					(unit 1)
 				)
@@
 		(dnp no)
 		(fields_autoplaced yes)
-		(property "Reference" "R93"
+		(property "Reference" "R37"
 			(at 156.21 68.58 0)
 			(show_name no)
@@
 			(project "pcb"
 				(path "/124991ae-9d31-41fe-b759-30be3a40922b/a13fb698-9f77-4d73-8ccf-806a48de5dab"
-					(reference "R93")
+					(reference "R37")
 					(unit 1)
 				)
