File: pcb/pcb.kicad_pcb (KiCad board)
At the start: 2 copper layers, 74 parts, among them J1 43045-0212, J2 XH_B4B, J3 XT60-M, Q1 BSS84K, Q2 BSS84K, Q3 BSS84K, Q8 SP30N16NJ, U1 INA219BxD, U2 MX27524ES, U3 MX27524ES, U4 EA8276P8R

Commit message: fixed schematic
Parts:
- removed FB7: 600@100MHz 100m, Inductor_SMD:L_0805_2012Metric
- removed Q8: SP30N16NJ, custom:PDFNWB-8L(3.3x3.3)
- added C32: 220uF 25V, Capacitor_SMD:CP_Elec_6.3x7.7, F.Cu at (39.2, 80.0)
- added C33: 10uF 25V, Capacitor_SMD:C_1206_3216Metric, F.Cu at (55.0, 89.4)
- added C34: 22pF 50V C0G, Capacitor_SMD:C_0402_1005Metric, F.Cu at (59.4, 57.4)
- added C35: 10uF 25V, Capacitor_SMD:C_1206_3216Metric, F.Cu at (55.0, 92.8)
- added C36: 220uF 25V, Capacitor_SMD:CP_Elec_6.3x7.7, F.Cu at (39.2, 88.2)
- added C37: 10uF 25V, Capacitor_SMD:C_1206_3216Metric, F.Cu at (55.0, 96.1)
- added C38: 10uF 16V A, Capacitor_Tantalum_SMD:CP_EIA-3216-18_Kemet-A, F.Cu at (87.3, 100.2)
- added C39: 1uF 25V, Capacitor_SMD:C_0603_1608Metric, F.Cu at (64.8, 99.8)
- added C40: 100nF 25V, Capacitor_SMD:C_0402_1005Metric, F.Cu at (59.4, 59.4)
- added C41: 100nF 25V, Capacitor_SMD:C_0402_1005Metric, F.Cu at (59.4, 61.3)
- added C42: 100nF 25V, Capacitor_SMD:C_0402_1005Metric, F.Cu at (59.4, 63.3)
- added C43: 2.2uF 6.3V, Capacitor_SMD:C_0402_1005Metric, F.Cu at (62.2, 51.5)
- added C44: 100nF 25V, Capacitor_SMD:C_0402_1005Metric, F.Cu at (62.2, 53.5)
- added C45: 100nF 25V, Capacitor_SMD:C_0402_1005Metric, F.Cu at (62.2, 55.4)
- added C46: 33pF 50V C0G, Capacitor_SMD:C_0402_1005Metric, F.Cu at (62.2, 57.4)
- added C47: 2.2uF 6.3V, Capacitor_SMD:C_0402_1005Metric, F.Cu at (62.2, 59.4)
- added C48: 100nF 25V, Capacitor_SMD:C_0402_1005Metric, F.Cu at (62.2, 61.3)
- added C49: 2.2uF 6.3V, Capacitor_SMD:C_0402_1005Metric, F.Cu at (62.2, 63.3)
- added C50: 100nF 25V, Capacitor_SMD:C_0402_1005Metric, F.Cu at (65.1, 51.5)
- added C51: 100nF 25V, Capacitor_SMD:C_0402_1005Metric, F.Cu at (65.1, 53.5)
- added C52: 100nF 25V, Capacitor_SMD:C_0402_1005Metric, F.Cu at (65.1, 55.4)
- added C53: 33pF 50V C0G, Capacitor_SMD:C_0402_1005Metric, F.Cu at (65.1, 57.4)
- added C54: 100nF 25V, Capacitor_SMD:C_0402_1005Metric, F.Cu at (65.1, 59.4)
- added D5: XL-1005SURC, LED_SMD:LED_0402_1005Metric, F.Cu at (50.7, 77.6)
- added F2: 4A 15V, Fuse:Fuse_1206_3216Metric, F.Cu at (72.3, 87.3)
- added FB1: 600@100MHz 100m, Inductor_SMD:L_0805_2012Metric, F.Cu at (73.5, 58.8)
- added FB2: 600@100MHz 100m, Inductor_SMD:L_0805_2012Metric, F.Cu at (73.5, 61.6)
- added J4: USB_A, Connector_USB:USB_A_Molex_67643_Horizontal, F.Cu at (39.6, 53.8)
- added J5: PinHeader_P2.54_01x04, Connector_PinHeader_2.54mm:PinHeader_1x04_P2.54mm_Vertical, F.Cu at (46.7, 70.1)
- added J6: USB_C_Receptacle_USB2.0_16P, custom:USB_C_Receptacle_16P, F.Cu at (39.8, 113.8)
- added Q4: SP30N16NJ, custom:PDFNWB-8L(3.3x3.3), F.Cu at (68.9, 60.0)
- added Q5: AO3400A, Package_TO_SOT_SMD:SOT-23, F.Cu at (60.3, 104.0)
- added R14: 200 1% 250mW, Resistor_SMD:R_1206_3216Metric, F.Cu at (72.3, 100.5)
- added R15: 2.2k 5%, Resistor_SMD:R_0201_0603Metric, F.Cu at (50.3, 70.4)
- added R16: 10k 5%, Resistor_SMD:R_0402_1005Metric, F.Cu at (62.2, 79.5)
- added R28: 1kR 1%, Resistor_SMD:R_0402_1005Metric, F.Cu at (65.1, 87.5)
- added R29: 10k 5%, Resistor_SMD:R_0402_1005Metric, F.Cu at (68.0, 75.5)
- added R30: 27 1%, Resistor_SMD:R_0603_1608Metric, F.Cu at (64.8, 102.3)
- added R31: 27 1%, Resistor_SMD:R_0603_1608Metric, F.Cu at (64.8, 104.8)
- added R32: 10k 5%, Resistor_SMD:R_0402_1005Metric, F.Cu at (68.0, 77.5)
- added R33: 1k 1%, Resistor_SMD:R_0402_1005Metric, F.Cu at (68.0, 79.5)
- added R34: 1k 1%, Resistor_SMD:R_0402_1005Metric, F.Cu at (68.0, 81.5)
- added R35: 2.2k 5%, Resistor_SMD:R_0201_0603Metric, F.Cu at (50.3, 73.9)
- added R36: 2.2k 5%, Resistor_SMD:R_0201_0603Metric, F.Cu at (50.3, 75.7)
- added R37: 5.1k 1%, Resistor_SMD:R_0402_1005Metric, F.Cu at (38.4, 119.5)
- added R38: 5.1k 1%, Resistor_SMD:R_0402_1005Metric, F.Cu at (38.4, 121.5)
- added SW1: TS-1088, Button_Switch_SMD:SW_SPST_TS-1088-xR020, F.Cu at (87.8, 52.8)
- added SW2: TS-1088, Button_Switch_SMD:SW_SPST_TS-1088-xR020, F.Cu at (87.8, 57.3)
- added U5: MX27524ES, Package_SO:Texas_DGN0008G_VSSOP-8-1EP_3x3mm_P0.65mm_EP2x2.94mm_Mask1.846x2.15mm_ThermalVias, F.Cu at (80.6, 57.5)
- added U6: W25Q16JVSS, Package_SO:SOIC-8_5.3x5.3mm_P1.27mm, F.Cu at (71.7, 54.0)
- added U7: RP2040, Package_DFN_QFN:QFN-56-1EP_7x7mm_P0.4mm_EP3.2x3.2mm, F.Cu at (79.8, 100.2)
- added U8: ESD73034D-10/TR(ES), Package_DFN_QFN:Diodes_UDFN-10_1x2.5mm_P0.5mm, F.Cu at (35.5, 120.6)
- added Y1: X322512MSB4SI, Crystal:Crystal_SMD_3225-4Pin_3.2x2.5mm, F.Cu at (87.0, 104.1)
- C1: value 220uF 25V -> 47uF 25V; footprint Capacitor_SMD:CP_Elec_6.3x7.7 -> Capacitor_SMD:C_Elec_6.3x5.4
- C14: value 100nF 25V -> 220uF 25V; footprint Capacitor_SMD:C_0402_1005Metric -> Capacitor_SMD:CP_Elec_6.3x7.7
- C15: value 220uF 25V -> 1uF 25V; footprint Capacitor_SMD:CP_Elec_6.3x7.7 -> Capacitor_SMD:C_0603_1608Metric
- C16, C21, C26, C27: value 10uF 25V -> 100nF 25V; footprint Capacitor_SMD:C_1206_3216Metric -> Capacitor_SMD:C_0402_1005Metric
- C18, C28, C29, C30: value 100nF 25V -> 10uF 25V; footprint Capacitor_SMD:C_0402_1005Metric -> Capacitor_SMD:C_1206_3216Metric
- C19: value 10uF 16V A -> 10uF 25V; footprint Capacitor_Tantalum_SMD:CP_EIA-3216-18_Kemet-A -> Capacitor_SMD:C_1206_3216Metric
- C2: value 220uF 25V -> 10uF 25V; footprint Capacitor_SMD:CP_Elec_6.3x7.7 -> Capacitor_SMD:C_1206_3216Metric
- C23, C24: value 1uF 25V -> 100nF 25V; footprint Capacitor_SMD:C_0603_1608Metric -> Capacitor_SMD:C_0402_1005Metric
- C25: value 1uF 25V -> 10uF 25V; footprint Capacitor_SMD:C_0603_1608Metric -> Capacitor_SMD:C_1206_3216Metric
- C31: value 22pF 50V C0G -> 100nF 25V
- C4: value 100nF 25V -> 10uF 16V A; footprint Capacitor_SMD:C_0402_1005Metric -> Capacitor_Tantalum_SMD:CP_EIA-3216-18_Kemet-A
- C5, C8: value 100nF 25V -> 1uF 25V; footprint Capacitor_SMD:C_0402_1005Metric -> Capacitor_SMD:C_0603_1608Metric
- C6: value 47uF 25V -> 100nF 25V; footprint Capacitor_SMD:C_Elec_6.3x5.4 -> Capacitor_SMD:C_0402_1005Metric
- C7: value 10uF 25V -> 1uF 25V; footprint Capacitor_SMD:C_1206_3216Metric -> Capacitor_SMD:C_0603_1608Metric
- D1: value SS34 -> SMF13CA; footprint Diode_SMD:D_SMA -> Diode_SMD:D_SOD-123F
- D4: value SMF13CA -> SS34; footprint Diode_SMD:D_SOD-123F -> Diode_SMD:D_SMA
- J1: value 43045-0212 -> XT60-M; footprint Connector_Molex:Molex_Micro-Fit_3.0_43045-0212_2x01_P3.00mm_Vertical -> Connector_AMASS:AMASS_XT60-M_1x02_P7.20mm_Vertical
- J3: value XT60-M -> 43045-0212; footprint Connector_AMASS:AMASS_XT60-M_1x02_P7.20mm_Vertical -> Connector_Molex:Molex_Micro-Fit_3.0_43045-0212_2x01_P3.00mm_Vertical
- L2: value 3.3uH -> 3.3uH 4.5A; footprint Inductor_SMD:L_Changjiang_FNR5030S -> Inductor_SMD:L_Bourns-SRN6028
- R1: value 200 1% 250mW -> 10m 1% 1W
- R10, R20: value 10k 5% -> 36k 5%
- R11, R9: value 36k 5% -> 10k 5%
- R13: value 10m 1% 1W -> 200 1% 250mW
- R17, R7: value 10k 5% -> 10 5%
- R21, R23: value 10 5% -> 10k 5%
- R22: value 10k 5% -> 2.2k 5%; footprint Resistor_SMD:R_0402_1005Metric -> Resistor_SMD:R_0201_0603Metric
- R25: value 10 5% -> 124k 1%
- R26: value 10 5% -> 22.1k 1%
- R3: value 200 1% 250mW -> 10 5%; footprint Resistor_SMD:R_1206_3216Metric -> Resistor_SMD:R_0402_1005Metric
- R4: value 2.2k 5% -> 10 5%; footprint Resistor_SMD:R_0201_0603Metric -> Resistor_SMD:R_0402_1005Metric
- R5: value 2.2k 5% -> 36k 5%; footprint Resistor_SMD:R_0201_0603Metric -> Resistor_SMD:R_0402_1005Metric
- R6: value 2.2k 5% -> 10k 5%; footprint Resistor_SMD:R_0201_0603Metric -> Resistor_SMD:R_0402_1005Metric
- R8: value 36k 5% -> 2.2k 5%; footprint Resistor_SMD:R_0402_1005Metric -> Resistor_SMD:R_0201_0603Metric
- U3: value MX27524ES -> TMI6050-33; footprint Package_SO:Texas_DGN0008G_VSSOP-8-1EP_3x3mm_P0.65mm_EP2x2.94mm_Mask1.846x2.15mm_ThermalVias -> Package_TO_SOT_SMD:SOT-23-5
- moved C4 800.6 mm to (87.3, 97.1)
- moved C1 797.2 mm to (80.4, 68.4)
- moved J3 796.4 mm to (88.2, 85.8)
- moved C15 792.0 mm to (64.8, 97.3)
- moved R1 790.8 mm to (72.3, 90.6)
- moved R2 790.8 mm to (72.3, 93.9)
- moved F1 788.9 mm to (72.3, 84.0)
- moved R13 788.9 mm to (72.3, 97.2)
- moved C8 778.7 mm to (64.8, 94.7)
- moved C5 776.9 mm to (64.8, 89.7)
- moved U3 776.6 mm to (86.5, 76.9)
- moved U1 773.5 mm to (79.3, 85.7)
- moved U4 773.5 mm to (79.3, 92.3)
- moved L1 773.0 mm to (42.5, 99.3)
- moved L2 770.9 mm to (89.3, 68.0)
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Connections:
- C10 pad 1: GND -> VCC
- C10 pad 2: VCC -> GND
- C11 pad 1: VCC -> /CELL1
- C13 pad 1: /CELL1_SENSE -> /BUCK_VB
- C14 pad 1: /CELL2_SENSE -> V_SOLAR
- C15 pad 1: V_SOLAR -> +5V
- C16 pad 1: V_SOLAR -> /CELL1_SENSE
- C17 pad 1: VCC -> /BUCK_SST
- C19 pad 1: /PSENSE_3.3VA -> +3.3V
- C2 pad 1: VCC -> V_SOLAR_PF
- C20 pad 1: /PSENSE_3.3VA -> V_SOLAR
- C21 pad 1: V_SOLAR_PF -> VCC
- C22 pad 1: /BUCK_BST -> /CELL2_SENSE
- C22 pad 2: /BUCK_SW -> GND
- C23 pad 1: /PSENSE_3.3VA -> GND
- C23 pad 2: GND -> VCC
- C24 pad 1: GND -> /BUCK_BST
- C24 pad 2: /PSENSE+ -> /BUCK_SW
- C25 pad 1: /PSENSE- -> VCC
- C27 pad 1: VCC -> GND
- C27 pad 2: GND -> VCC
- C29 pad 1: /BUCK_SST -> VCC
- C30 pad 1: /BUCK_VB -> +5V
- C31 pad 1: unconnected-(C31-Pad1) -> VCC
- C31 pad 2: /BUCK_FB -> GND
- C4 pad 1: /CELL2 -> /PSENSE_3.3VA
- C5 pad 1: /CELL1 -> /PSENSE_3.3VA
- C6 pad 1: VCC -> /CELL2
- C7 pad 1: VCC -> GND
- C7 pad 2: GND -> /PSENSE+
- C8 pad 1: VCC -> /PSENSE-
- C9 pad 1: GND -> /PSENSE_3.3VA
- C9 pad 2: VCC -> GND
- D1 pad 1: VCC -> GND
- D1 pad 2: Net-(D1-A) -> VCC_RAW
- D2 pad 2: VCC_RAW -> /CELL2
- D3 pad 2: /CELL2 -> /CELL1
- D4 pad 1: GND -> VCC
- D4 pad 2: /CELL1 -> Net-(D4-A)
- J1 pad 2: V_SOLAR_PF -> VCC_RAW
- J3 pad 2: VCC_RAW -> V_SOLAR_PF
- L1 pad 2: Net-(D1-A) -> Net-(D4-A)
- L2 pad 1: unconnected-(L2-Pad1) -> /BUCK_SW
- L2 pad 2: unconnected-(L2-Pad2) -> +5V
- R1 pad 1: Net-(Q1-D) -> V_SOLAR_PF
- R1 pad 2: GND -> V_SOLAR
- R10 pad 1: /CELL1_PF -> /CELL1
- R10 pad 2: GND -> /CELL1_PF
- R11 pad 1: /CELL2 -> /CELL1_PF
- R11 pad 2: /CELL2_PF -> GND
- R12 pad 1: /CELL2_PF -> VCC
- R12 pad 2: GND -> /BUCK_RUN
- R13 pad 1: V_SOLAR_PF -> Net-(Q2-D)
- R13 pad 2: V_SOLAR -> GND
- R17 pad 2: GND -> /BOOST_GATE
- R18 pad 1: /BOOST_GATE_DRV -> /CELL2_GATE_DRV
- R18 pad 2: /BOOST_GATE -> /CELL2_GATE
- R19 pad 1: /CELL1_GATE_DRV -> /CELL3_GATE_DRV
- R19 pad 2: /CELL1_GATE -> /CELL3_GATE
- R2 pad 1: Net-(Q2-D) -> Net-(Q1-D)
- R20 pad 1: /CELL1 -> /CELL2
- R20 pad 2: /CELL1_GATE_DRV -> /CELL2_PF
- R21 pad 1: /CELL2_GATE_DRV -> /CELL2_PF
- R21 pad 2: /CELL2_GATE -> GND
- R22 pad 1: /CELL2 -> /CELL2_PF
- R22 pad 2: /CELL2_GATE_DRV -> /CELL2_SENSE
- R23 pad 1: /CELL3_GATE_DRV -> /CELL2
- R23 pad 2: /CELL3_GATE -> /CELL2_GATE_DRV
- R25 pad 1: V_SOLAR_PF -> +5V
- R25 pad 2: /PSENSE+ -> /BUCK_FB
- R26 pad 1: V_SOLAR -> /BUCK_FB
- R26 pad 2: /PSENSE- -> GND
- R27 pad 1: VCC -> +3.3V
- R27 pad 2: /BUCK_RUN -> /QSPI_SS
- R3 pad 1: Net-(Q3-D) -> V_SOLAR_PF
- R3 pad 2: GND -> /PSENSE+
- R4 pad 1: /BATT_PF -> V_SOLAR
- R4 pad 2: /BATT_SENSE -> /PSENSE-
- R5 pad 1: /CELL1_PF -> VCC
- R5 pad 2: /CELL1_SENSE -> /BATT_PF
- R6 pad 1: /CELL2_PF -> /BATT_PF
- R6 pad 2: /CELL2_SENSE -> GND
- R7 pad 1: /BATT_PF -> /CELL1_GATE_DRV
- R7 pad 2: GND -> /CELL1_GATE
- R8 pad 1: VCC -> /BATT_PF
- R8 pad 2: /BATT_PF -> /BATT_SENSE
- R9 pad 2: /CELL1_PF -> /CELL1_GATE_DRV
- U3 pad 1: /CELL2_EN -> +5V
- U3 pad 2: /~{CELL2_SW} -> GND
- U3 pad 3: GND -> +5V
- U3 pad 4: /~{CELL3_SW} -> unconnected-(U3-NC-Pad4)
- U3 pad 5: /CELL3_GATE_DRV -> +3.3V
- U4 pad 5: (no net) -> GND
- U4 pad 6: (no net) -> /BUCK_SW
- U4 pad 8: GND -> VCC

Commit message: pcb done
Parts:
- removed C1: 47uF 25V, Capacitor_SMD:C_Elec_6.3x5.4
- removed C3: 100nF 25V, Capacitor_SMD:C_0402_1005Metric
- removed Q4: SP30N16NJ, custom:PDFNWB-8L(3.3x3.3)
- removed Q5: AO3400A, Package_TO_SOT_SMD:SOT-23
- added C55: 100nF 25V, Capacitor_SMD:C_0402_1005Metric, F.Cu at (-32.0, -21.8)
- added H1: M3, MountingHole:MountingHole_3.2mm_M3_Pad_Via, F.Cu at (-36.0, 26.0)
- added H2: M3, MountingHole:MountingHole_3.2mm_M3_Pad_Via, F.Cu at (13.0, -36.0)
- added H3: M3, MountingHole:MountingHole_3.2mm_M3_Pad_Via, F.Cu at (13.0, 26.0)
- added Q6: PTQ3060, custom:PDFNWB-8L(3.3x3.3), F.Cu at (-9.60, -21.6)
- added Q7: PTQ3060, custom:PDFNWB-8L(3.3x3.3), F.Cu at (-19.4, 18.8)
- R15, R22, R35, R36, R8: footprint Resistor_SMD:R_0201_0603Metric -> Resistor_SMD:R_0402_1005Metric
- R30, R31: footprint Resistor_SMD:R_0603_1608Metric -> Resistor_SMD:R_0402_1005Metric
- U6: value W25Q16JVSS -> W25Q16JVUXIQ; footprint Package_SO:SOIC-8_5.3x5.3mm_P1.27mm -> Package_SON:Winbond_USON-8-1EP_3x2mm_P0.5mm_EP0.2x1.6mm
- moved J3 166.7 mm to (-25.2, -36.4)
- moved C4 156.9 mm to (-9.44, -26.5), turned to -90 degrees
- moved R1 152.8 mm to (-16.2, -33.9)
- moved C8 148.8 mm to (-14.6, -31.1)
- moved C7 148.4 mm to (-17.8, -31.1)
- moved F1 148.0 mm to (-27.6, -25.2)
- moved U1 146.5 mm to (-14.8, -26.5), turned to 90 degrees
- moved R2 143.1 mm to (-36.4, 0.80)
- moved J1 142.7 mm to (-34.6, -34.6), turned to -90 degrees
- moved R13 141.9 mm to (-31.8, 0.80)
- moved J2 141.7 mm to (-36.4, -12.2), turned to 90 degrees
- moved R14 140.9 mm to (-27.2, 0.80)
- moved C5 139.5 mm to (-11.2, -27.3), turned to -90 degrees
- moved Y1 137.9 mm to (-13.0, 9.20), turned to 90 degrees
- moved Q3 134.8 mm to (-27.8, -2.40), turned to -90 degrees
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Connections:
- J2 pad 1: VCC_RAW -> GND
- J2 pad 2: /CELL2 -> /CELL1
- J2 pad 3: /CELL1 -> /CELL2
- J2 pad 4: GND -> VCC_RAW
- J5 pad 2: /SWCLK -> /NRST
- J5 pad 3: /SWDIO -> /SWCLK
- J5 pad 4: /NRST -> /SWDIO
- R13 pad 2: GND -> /CELL1
- R14 pad 2: GND -> /CELL2
- R30 pad 1: /USB_D+ -> /USB_D-
- R31 pad 1: /USB_D- -> /USB_D+
- U2 pad 4: /~{CELL1_SW} -> /~{CELL3_SW}
- U2 pad 5: /CELL1_GATE_DRV -> /CELL3_GATE_DRV
- U2 pad 8: /CELL1_EN -> /CELL3_EN
- U5 pad 4: /~{CELL3_SW} -> /~{CELL1_SW}
- U5 pad 5: /CELL3_GATE_DRV -> /CELL1_GATE_DRV
- U5 pad 8: /CELL3_EN -> /CELL1_EN
- U7 pad 11: /~{CELL3_SW} -> /CELL1_EN
- U7 pad 12: /CELL3_EN -> /~{CELL1_SW}
- U7 pad 13: /USB_PWRON -> /~{CELL2_SW}
- U7 pad 14: /~{LED} -> /CELL2_EN
- U7 pad 35: unconnected-(U7-GPIO23-Pad35) -> /~{LED}
- U7 pad 39: /CELL1_SENSE -> /CELL2_SENSE
- U7 pad 4: /BOOST_SW -> /CELL3_EN
- U7 pad 40: /CELL2_SENSE -> /CELL1_SENSE
- U7 pad 41: unconnected-(U7-GPIO29/ADC3-Pad41) -> /USB_PWRON
- U7 pad 5: /BOOST_EN -> /~{CELL3_SW}
- U7 pad 6: /~{CELL1_SW} -> /BOOST_SW
- U7 pad 7: /CELL1_EN -> /BOOST_EN
- U7 pad 8: /CELL2_EN -> unconnected-(U7-GPIO6-Pad8)
- U7 pad 9: /~{CELL2_SW} -> unconnected-(U7-GPIO7-Pad9)
Routing:
- net GND: track 0.00 -> 344.8 mm, vias 0 -> 161
- net +3.3V: track 0.00 -> 121.7 mm, vias 0 -> 5
- net /SDA: track 0.00 -> 92.5 mm, vias 0 -> 4
- net VCC: track 0.00 -> 91.8 mm, vias 0 -> 2
- net /SCL: track 0.00 -> 91.6 mm, vias 0 -> 4
- net +5V: track 0.00 -> 84.1 mm, vias 0 -> 6
- net /BOOST_EN: track 0.00 -> 54.8 mm, vias 0 -> 2
- net /BOOST_SW: track 0.00 -> 54.1 mm, vias 0 -> 2
- net /~{CELL3_SW}: track 0.00 -> 51.5 mm, vias 0 -> 2
- net /CELL3_EN: track 0.00 -> 45.7 mm, vias 0 -> 4
- net VCC_RAW: track 0.00 -> 43.5 mm
- net Net-(D4-A): track 0.00 -> 43.4 mm
- net /CELL1_SENSE: track 0.00 -> 41.7 mm
- net /CELL2_SENSE: track 0.00 -> 36.2 mm
- net /CELL2: track 0.00 -> 32.2 mm, vias 0 -> 2
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- added copper zone on B.Cu, net GND
- added copper zone on F.Cu, net GND
Other:
- board outline added: 57 x 70 mm
- board text added: "BOOT"
- board text added: "RST"

Commit message: fixed some issues
Parts:
- removed C8: 1uF 25V, Capacitor_SMD:C_0603_1608Metric
- removed R23, R24, R9: 10k 5%, Resistor_SMD:R_0402_1005Metric
- added R39: 10k 5%, Resistor_SMD:R_0402_1005Metric, F.Cu at (-14.8, 3.60)
- added R40: 10k 5%, Resistor_SMD:R_0402_1005Metric, F.Cu at (-13.8, 3.60)
- added R41: 10k 5%, Resistor_SMD:R_0402_1005Metric, F.Cu at (-8.00, 4.60)
- added R42: 10k 5%, Resistor_SMD:R_0402_1005Metric, F.Cu at (-8.00, 3.60)
- added R43: 10k 5%, Resistor_SMD:R_0402_1005Metric, F.Cu at (-1.20, -13.8)
- added R44: 10k 5%, Resistor_SMD:R_0402_1005Metric, F.Cu at (-3.60, -13.8)
- moved C7 1.64 mm to (-16.2, -31.0), turned to 180 degrees
Connections:
- C7 pad 1: GND -> /PSENSE-
Routing:
- net +3.3V: track 121.7 -> 139.7 mm, vias 5 -> 7
- net GND: track 344.8 -> 340.5 mm, vias 161 -> 159
- net /~{CELL2_SW}: track 21.5 -> 25.3 mm, vias 0 -> 2
- net /CELL2_EN: track 21.6 -> 25.2 mm, vias 0 -> 2
- net /~{CELL3_SW}: track 51.5 -> 54.8 mm, vias 2 -> 4
- net /~{CELL1_SW}: track 20.3 -> 23.3 mm, vias 0 -> 2
- net /CELL1_EN: track 27.9 -> 29.5 mm
- net /CELL2_GATE_DRV: track 9.05 -> 8.12 mm
- net /CELL1_GATE_DRV: track 15.7 -> 14.8 mm
- net /CELL3_GATE_DRV: track 17.5 -> 16.5 mm
- net /CELL3_EN: track 45.7 -> 46.5 mm
- net /CELL2: track 32.2 -> 31.4 mm
- net /CELL1: track 28.7 -> 28.1 mm
