File: pcb/pcb.kicad_sch (KiCad schematic)
At the start: 117 parts, among them J1 43045-0212, J2 XH_B4B, J3 XT60-M, J4 USB_A, J5 PinHeader_P2.54_01x04, Q1 BSS84K, Q2 BSS84K, Q3 BSS84K, Q4 AO3400A, Q8 SP30N16NJ, SW1 TS-1088, SW2 TS-1088, U1 INA219BxD, U2 MX27524ES, U3 MX27524ES, U4 EA8276P8R, U5 TMI6050-33, U6 RP2040, U7 W25Q16JVSS, Y1 X322512MSB4SI

Commit message: fixed schematic
Parts:
- removed C39: 10uF 16V A, Capacitor_Tantalum_SMD:CP_EIA-3216-18_Kemet-A, symbol Device:C_Polarized
- removed C44, C59, C60: 100nF 25V, Capacitor_SMD:C_0402_1005Metric, symbol Device:C
- removed C61, C62: 2.2uF 6.3V, Capacitor_SMD:C_0402_1005Metric, symbol Device:C
- removed FB8: 600@100MHz 100m, Inductor_SMD:L_0805_2012Metric, symbol Device:FerriteBead
- removed R28, R29: 27 1%, Resistor_SMD:R_0603_1608Metric, symbol Device:R
- removed U6: RP2040, Package_DFN_QFN:QFN-56-1EP_7x7mm_P0.4mm_EP3.2x3.2mm, symbol MCU_RaspberryPi:RP2040
- removed U7: W25Q16JVSS, Package_SON:Winbond_USON-8-1EP_3x2mm_P0.5mm_EP0.2x1.6mm, symbol Memory_Flash:W25Q16JVSS
- added C38: 10uF 16V A, Capacitor_Tantalum_SMD:CP_EIA-3216-18_Kemet-A, symbol Device:C_Polarized
- added C39: 1uF 25V, Capacitor_SMD:C_0603_1608Metric, symbol Device:C
- added C41, C50, C52: 100nF 25V, Capacitor_SMD:C_0402_1005Metric, symbol Device:C
- added C49: 2.2uF 6.3V, Capacitor_SMD:C_0402_1005Metric, symbol Device:C
- added D5: XL-1005SURC, LED_SMD:LED_0402_1005Metric, symbol Device:LED
- added FB2: 600@100MHz 100m, Inductor_SMD:L_0805_2012Metric, symbol Device:FerriteBead
- added R30: 27 1%, Resistor_SMD:R_0603_1608Metric, symbol Device:R
- added R32: 10k 5%, Resistor_SMD:R_0402_1005Metric, symbol Device:R
- added R34: 1k 1%, Resistor_SMD:R_0402_1005Metric, symbol Device:R
- added R35, R36: 2.2k 5%, Resistor_SMD:R_0201_0603Metric, symbol Device:R
- added U6: W25Q16JVSS, Package_SO:SOIC-8_5.3x5.3mm_P1.27mm, symbol Memory_Flash:W25Q16JVSS
- added U7: RP2040, Package_DFN_QFN:QFN-56-1EP_7x7mm_P0.4mm_EP3.2x3.2mm, symbol MCU_RaspberryPi:RP2040
- C43: value 1uF 25V -> 2.2uF 6.3V; footprint Capacitor_SMD:C_0603_1608Metric -> Capacitor_SMD:C_0402_1005Metric; MPN 0603B105M250NT -> 0402B104K250NT
- R31: value 10k 5% -> 27 1%; footprint Resistor_SMD:R_0402_1005Metric -> Resistor_SMD:R_0603_1608Metric
- R33: value 1kR 1% -> 1k 1%
- renumbered C6 to C1, C8 to C10, C5 to C11, C30 to C13, C15 to C14, C36 to C15, C13 to C16, C29 to C17, C16 to C18, C37 to C19, C21 to C2, C18 to C20, C28 to C21, C14 to C22, C9 to C23, C22 to C24, C26 to C25, C17 to C26, C10 to C27, C27 to C28, C7 to C29, C32 to C30, C11 to C31, C1 to C32, C31 to C34, C34 to C35, C2 to C36, C35 to C37, C19 to C4, C53 to C40, C54 to C42, C63 to C44, C55 to C45, C38 to C46, C64 to C47, C56 to C48, C23 to C5, C57 to C51, C40 to C53, C58 to C54, C4 to C6, C24 to C7, C25 to C8, C20 to C9, D2 to D1, D3 to D2, D4 to D3, D1 to D4, FB7 to FB1, J3 to J1, J1 to J3, Q8 to Q4, Q4 to Q5, R13 to R1, R9 to R10, R10 to R11, R27 to R12, R2 to R13, R3 to R14, R5 to R15, R17 to R16, R18 to R17, R21 to R18, R23 to R19, R1 to R2, R11 to R20, R12 to R21, R6 to R22, R22 to R23, R14 to R25, R15 to R26, R32 to R27, R30 to R28, R34 to R29, R25 to R3, R26 to R4, R8 to R5, R7 to R6, R19 to R7, R4 to R8, R20 to R9, U5 to U3, U3 to U5
Connections:
- net +1V1: now also C49.1, C50.1, C52.1, U7.23 (DVDD), U7.45 (VREG_VOUT), U7.50 (DVDD)
- net +3.3V: now also C43.1, FB2.1, R32.1, R34.1, R35.2, R36.2, U6.8 (VCC), U7.1 (IOVDD), U7.10 (IOVDD), U7.22 (IOVDD), U7.33 (IOVDD), U7.42 (IOVDD), U7.44 (VREG_VIN), U7.48 (USB_VDD), U7.49 (IOVDD); no longer R31.1
- net BATT_SENSE: now also U7.38 (GPIO26/ADC0)
- net BOOST_EN: now also U7.5 (GPIO3)
- net BOOST_SW: now also U7.4 (GPIO2)
- net BUCK_SW: now also U4.6 (SW); no longer U4. (SW)
- net CELL1_EN: now also U7.7 (GPIO5)
- net CELL1_SENSE: now also U7.39 (GPIO27/ADC1)
- net CELL2_EN: now also U7.8 (GPIO6)
- net CELL2_SENSE: now also U7.40 (GPIO28/ADC2)
- net CELL3_EN: now also U7.12 (GPIO9)
- net GND: now also U4.5 (GND), C38.2, C39.2, C41.2, C49.2, C50.2, C52.2, U6.4 (GND), U7.19 (TESTEN), U7.57 (GND); no longer U4.8 (GND)
- net MCU_3.3VA: now also C38.1, C39.1, C41.1, FB2.2, U7.43 (ADC_AVDD); no longer C43.1
- net NRST: now also R32.2, U7.26 (RUN); no longer R31.2
- net QSPI_SCLK: now also U6.6 (CLK), U7.52 (QSPI_SCLK)
- net QSPI_SD0: now also U6.5 (DI/IO_{0}), U7.53 (QSPI_SD0)
- net QSPI_SD1: now also U6.2 (DO/IO_{1}), U7.55 (QSPI_SD1)
- net QSPI_SD2: now also U6.3 (~{WP}/IO_{2}), U7.54 (QSPI_SD2)
- net QSPI_SD3: now also U6.7 (~{HOLD}/~{RESET}/IO_{3}), U7.51 (QSPI_SD3)
- net QSPI_SS: now also U6.1 (~{CS}), U7.56 (~{QSPI_SS})
- net SCL: now also R36.1, U7.3 (GPIO1)
- net SDA: now also R35.1, U7.2 (GPIO0)
- net SWCLK: now also U7.24 (SWCLK)
- net SWDIO: now also U7.25 (SWDIO)
- net USB_D+: now also R30.1
- net USB_D-: now also R31.1
- net USB_PWRON: now also U7.13 (GPIO10)
- net XIN: now also U7.20 (XIN)
- net XOUT: now also U7.21 (XOUT)
- net ~{CELL1_SW}: now also U7.6 (GPIO4)
- net ~{CELL2_SW}: now also U7.9 (GPIO7)
- net ~{CELL3_SW}: now also U7.11 (GPIO8)
- new net: R31.2, U7.47 (USB_DP)
- new net: R30.2, U7.46 (USB_DM)
- new net LED_MID: D5.2 (A), R34.2
- new net ~{LED}: D5.1 (K), U7.14 (GPIO11)
- no-connect marks 2 -> 17
Other:
- moved on the sheet: J5

Commit message: pcb done
Parts:
- removed C1: 47uF 25V, Capacitor_SMD:C_Elec_6.3x5.4, symbol Device:C_Polarized
- removed C3: 100nF 25V, Capacitor_SMD:C_0402_1005Metric, symbol Device:C
- removed Q4: SP30N16NJ, custom:PDFNWB-8L(3.3x3.3), symbol Custom:SP30N16NJ
- removed Q5: AO3400A, Package_TO_SOT_SMD:SOT-23, symbol Transistor_FET:AO3400A
- removed U6: W25Q16JVSS, Package_SO:SOIC-8_5.3x5.3mm_P1.27mm, symbol Memory_Flash:W25Q16JVSS
- added C55: 100nF 25V, Capacitor_SMD:C_0402_1005Metric, symbol Device:C
- added H1, H2, H3: M3, MountingHole:MountingHole_3.2mm_M3_Pad_Via, symbol Mechanical:MountingHole_Pad
- added Q6, Q7: PTQ3060, custom:PDFNWB-8L(3.3x3.3), symbol Custom:PTQ3060
- added U6: W25Q16JVUXIQ, Package_SON:Winbond_USON-8-1EP_3x2mm_P0.5mm_EP0.2x1.6mm, symbol Custom:W25Q16JVUXIQ
- R15, R22, R35, R36, R8: footprint Resistor_SMD:R_0201_0603Metric -> Resistor_SMD:R_0402_1005Metric
- R30, R31: footprint Resistor_SMD:R_0603_1608Metric -> Resistor_SMD:R_0402_1005Metric
Connections:
- net +3.3V: now also U6.8 (VCC)
- net BOOST_EN: now also U7.7 (GPIO5); no longer U7.5 (GPIO3)
- net BOOST_GATE: now also Q6.2 (G)
- net BOOST_SW: now also U7.6 (GPIO4); no longer U7.4 (GPIO2)
- net CELL1: now also J2.2 (Pin_2), R13.2; no longer J2.3 (Pin_3)
- net CELL1_EN: now also U5.8 (ENB), U7.11 (GPIO8); no longer U2.8 (ENB), U7.7 (GPIO5)
- net CELL1_GATE_DRV: now also U5.5 (OUTB); no longer U2.5 (OUTB)
- net CELL1_SENSE: now also U7.40 (GPIO28/ADC2); no longer U7.39 (GPIO27/ADC1)
- net CELL2: now also J2.3 (Pin_3), R14.2; no longer J2.2 (Pin_2)
- net CELL2_EN: now also U7.14 (GPIO11); no longer U7.8 (GPIO6)
- net CELL2_SENSE: now also U7.39 (GPIO27/ADC1); no longer U7.40 (GPIO28/ADC2)
- net CELL3_EN: now also U2.8 (ENB), U7.4 (GPIO2); no longer U5.8 (ENB), U7.12 (GPIO9)
- net CELL3_GATE_DRV: now also U2.5 (OUTB); no longer U5.5 (OUTB)
- net GND: now also J2.1 (Pin_1), C55.2, Q6.1 (S), Q7.1 (S), U6.4 (GND), U6.9 (EP); no longer J2.4 (Pin_4), R13.2, R14.2
- net NRST: now also J5.2 (Pin_2); no longer J5.4 (Pin_4)
- net QSPI_SCLK: now also U6.6 (CLK)
- net QSPI_SD0: now also U6.5 (DI/IO_{0})
- net QSPI_SD1: now also U6.2 (DO/IO_{1})
- net QSPI_SD2: now also U6.3 (~{WP}/IO_{2})
- net QSPI_SD3: now also U6.7 (~{HOLD}/~{RESET}/IO_{3})
- net QSPI_SS: now also U6.1 (~{CS})
- net SWCLK: now also J5.3 (Pin_3); no longer J5.2 (Pin_2)
- net SWDIO: now also J5.4 (Pin_4); no longer J5.3 (Pin_3)
- net USB_D+: now also R31.1; no longer R30.1
- net USB_D-: now also R30.1; no longer R31.1
- net USB_LOW_PFUSE: now also Q7.3 (D)
- net USB_PWRON: now also U7.41 (GPIO29/ADC3); no longer U7.13 (GPIO10)
- net VCC_RAW: now also J2.4 (Pin_4), C55.1; no longer J2.1 (Pin_1)
- net ~{CELL1_SW}: now also U5.4 (INB), U7.12 (GPIO9); no longer U2.4 (INB), U7.6 (GPIO4)
- net ~{CELL2_SW}: now also U7.13 (GPIO10); no longer U7.9 (GPIO7)
- net ~{CELL3_SW}: now also U2.4 (INB), U7.5 (GPIO3); no longer U5.4 (INB), U7.11 (GPIO8)
- net ~{LED}: now also U7.35 (GPIO23); no longer U7.14 (GPIO11)
- net at D4.2 (A), L1.2: now also Q6.3 (D)
- net at R33.2: now also Q7.2 (G)
- no-connect marks 17 -> 20
Other:
- note added: "MOUNT"
- note added: "designing for output = 12.6V, 2A: inductor ripple current (using 20%) = 0.84A at 150kHz, L = 25.3uH (pick 33uH) at input = 5V (min), output = 13V (12.6 + diode): duty cycle ~= 0.7 ripple current ~= 0.71A peak inductor current ~= 7A 2x 220uF, 35mOhm(@100kHz) polymer caps yields ~150mV ripple RC filter cell voltage sensing 15nC gate charge at ~1A: 15ns @2A, 150kHz: switching losses ~= 0.1W, conduct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"
- note added: "~3.6W losses @2A ~88% efficiency"
- note removed: "designing for output = 12.6V, 2A: inductor ripple current (using 20%) = 0.84A at 150kHz, L = 25.3uH (pick 33uH) at input = 5V (min), output = 13V (12.6 + diode): duty cycle ~= 0.7 ripple current ~= 0.71A peak inductor current ~= 7A 2x 220uF, 35mOhm(@100kHz) polymer caps yields ~150mV ripple RC filter cell voltage sensing 5nC gate charge at ~1A: 5ns @2A, 150kHz: switching losses ~= 30mW, conductio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"
- note removed: "~4W losses @2A ~86% efficiency"
- moved on the sheet: D1, F1

Commit message: fixed some issues
Parts:
- removed C8: 1uF 25V, Capacitor_SMD:C_0603_1608Metric, symbol Device:C
- removed R23, R24, R9: 10k 5%, Resistor_SMD:R_0402_1005Metric, symbol Device:R
- added R39, R40, R41, R42, R43, R44: 10k 5%, Resistor_SMD:R_0402_1005Metric, symbol Device:R
Connections:
- net +3.3V: now also R39.1, R40.1, R41.1, R42.1, R43.1, R44.1
- net CELL1_EN: now also R39.2
- net CELL2_EN: now also R41.2
- net CELL3_EN: now also R43.2
- net GND: no longer C7.1
- net PSENSE-: now also C7.1
- net ~{CELL1_SW}: now also R40.2
- net ~{CELL2_SW}: now also R42.2
- net ~{CELL3_SW}: now also R44.2
Other:
- note added: "16kHz LPF"
- note removed: "100kHz LPF"
- moved on the sheet: C31, U5
